File: hardware/front.brd (EAGLE design)
At the start: 119.2 x 60.4 mm, 22 parts

Commit message: pdf fuer die kicadler
Changed lines of the file:
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@@
 <?xml version="1.0" encoding="utf-8"?>
 <!DOCTYPE eagle SYSTEM "eagle.dtd">
-<eagle version="6.2">
+<eagle version="6.6.0">
 <drawing>
 <settings>
@@
 </class>
 </classes>
-<designrules>
+<designrules name="default">
 <description language="de">&lt;b&gt;EAGLE Design Rules&lt;/b&gt;
 &lt;p&gt;
@@
 <signal name="GND">
 <polygon width="0.4064" layer="16" isolate="0.4064">
-<vertex x="-11.049" y="98.7425"/>
-<vertex x="156.718" y="98.7425"/>
-<vertex x="156.718" y="7.874"/>
-<vertex x="-11.049" y="7.874"/>
+<vertex x="16.3195" y="84.201"/>
+<vertex x="141.6685" y="83.312"/>
+<vertex x="140.7795" y="16.7005"/>
+<vertex x="15.4305" y="17.5895"/>
 </polygon>
 <contactref element="LED3" pad="K"/>
