File: hardware/controller.brd (EAGLE design)
At the start: 123.8 x 63.2 mm, 42 parts, among them IC1 MEGA8-AI, IC2 MAX232ECWE, K1 G5LE, X1 MSTBA5

Commit message: pdf fuer die kicadler
Parts:
- moved C1 43.0 mm to (38.7, 18.4)
- moved C10 43.0 mm to (33.7, 43.8)
- moved C11 43.0 mm to (58.4, 45.1)
- moved C12 43.0 mm to (8.89, 26.7)
- moved C13 43.0 mm to (58.4, 31.8)
- moved C14 43.0 mm to (57.8, 20.3)
- moved C3 43.0 mm to (5.08, 38.7)
- moved C4 43.0 mm to (4.45, 34.3)
- moved C5 43.0 mm to (4.45, 31.1)
- moved C7 43.0 mm to (17.8, 38.7)
- moved C8 43.0 mm to (57.8, 20.3)
- moved D1 43.0 mm to (61.0, 52.1)
- moved D2 43.0 mm to (61.0, 48.9)
- moved D3 43.0 mm to (61.0, 35.6)
- moved D4 43.0 mm to (61.0, 38.7)
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
Commit message: minor pcb changes
Parts:
- added D5: 1N4148DO35-10, diode:DO35-10
Connections:
- net +5V: now also D5.C
- net N$37: now also D5.A
Changed lines of the file:
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@@
 <layer number="97" name="Info" color="7" fill="1" visible="no" active="no"/>
 <layer number="98" name="Guide" color="6" fill="1" visible="no" active="no"/>
+<layer number="99" name="SpiceOrder" color="5" fill="1" visible="no" active="no"/>
 </layers>
 <board>
@@
 <wire x1="123.805" y1="63.17" x2="0" y2="63.17" width="0" layer="20"/>
 <wire x1="0" y1="63.17" x2="0" y2="0" width="0" layer="20"/>
-<polygon width="1.9304" layer="41">
-<vertex x="75.565" y="61.595"/>
-<vertex x="128.27" y="61.595"/>
-<vertex x="128.27" y="19.685"/>
-<vertex x="75.565" y="19.685"/>
-</polygon>
-<polygon width="1.9304" layer="42">
-<vertex x="75.565" y="61.595"/>
-<vertex x="128.27" y="61.595"/>
-<vertex x="128.27" y="20.32"/>
-<vertex x="75.565" y="20.32"/>
-</polygon>
 </plain>
 <attributes>
@@
 <element name="JP3" library="pinhead" package="1X04" value="" x="17.78" y="51.435" rot="R180"/>
 <element name="JP7" library="pinhead" package="1X04" value="" x="30.48" y="51.435" rot="R180"/>
+<element name="D5" library="diode" package="DO35-10" value="1N4148DO35-10" x="71.12" y="9.525" rot="R270"/>
 </elements>
 <signals>
@@
 <polygon width="0.4064" layer="16" isolate="0.4064">
 <vertex x="-3.81" y="64.77"/>
-<vertex x="127.635" y="65.405"/>
-<vertex x="127.635" y="-1.905"/>
+<vertex x="69.215" y="63.5"/>
+<vertex x="69.215" y="-3.81"/>
 <vertex x="-3.81" y="-3.175"/>
 </polygon>
 <polygon width="0.4064" layer="1" isolate="0.4064">
 <vertex x="-3.81" y="64.77"/>
-<vertex x="127.635" y="64.77"/>
-<vertex x="127.635" y="-3.175"/>
+<vertex x="69.215" y="64.135"/>
+<vertex x="69.215" y="-3.81"/>
 <vertex x="-3.81" y="-3.175"/>
 </polygon>
@@
 <wire x1="20.955" y1="23.495" x2="20.955" y2="24.765" width="0.4064" layer="1"/>
 <wire x1="53.975" y1="20.32" x2="56.835" y2="20.32" width="0.4064" layer="1"/>
-<wire x1="79.502" y1="14.859" x2="55.626" y2="14.859" width="0.4064" layer="1"/>
-<wire x1="55.626" y1="14.859" x2="53.975" y2="16.51" width="0.4064" layer="1"/>
-<wire x1="53.975" y1="16.51" x2="53.975" y2="20.32" width="0.4064" layer="1"/>
+<wire x1="79.502" y1="14.859" x2="71.12" y2="14.859" width="0.6096" layer="1"/>
+<wire x1="71.12" y1="14.859" x2="55.626" y2="14.859" width="0.6096" layer="1"/>
+<wire x1="55.626" y1="14.859" x2="53.975" y2="16.51" width="0.6096" layer="1"/>
+<wire x1="53.975" y1="16.51" x2="53.975" y2="20.32" width="0.6096" layer="1"/>
+<contactref element="D5" pad="C"/>
+<wire x1="71.12" y1="14.605" x2="71.12" y2="14.859" width="0.6096" layer="1"/>
 <wire x1="10.16" y1="26.67" x2="9.84" y2="26.67" width="0" layer="19" extent="1-1"/>
 </signal>
@@
 <contactref element="K1" pad="1"/>
 <wire x1="79.502" y1="2.921" x2="79.502" y2="3.048" width="0.4064" layer="1"/>
-<wire x1="79.502" y1="3.048" x2="78.105" y2="4.445" width="0.4064" layer="1"/>
-<wire x1="78.105" y1="4.445" x2="60.325" y2="4.445" width="0.4064" layer="1"/>
+<wire x1="79.502" y1="3.048" x2="78.105" y2="4.445" width="0.6096" layer="1"/>
+<wire x1="78.105" y1="4.445" x2="72.39" y2="4.445" width="0.6096" layer="1"/>
+<contactref element="D5" pad="A"/>
+<wire x1="71.12" y1="4.445" x2="60.325" y2="4.445" width="0.6096" layer="1"/>
+<wire x1="71.12" y1="4.445" x2="72.39" y2="4.445" width="0.6096" layer="1"/>
 </signal>
 </signals>
