File: hardware/controller.sch (EAGLE design)
At the start: 42 parts, among them IC1 MEGA8-AI, IC2 MAX232ECWE, K1 G5LE, X1 MSTBA5

Commit message: pdf fuer die kicadler
Other:
- moved on the sheet: C11, C13, C14, C3, C4, C5, C6, D1, D2, D3, D4, H1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

Commit message: minor pcb changes
Parts:
- added D5: 1N4148DO35-10, diode:1N4148DO35-10
Connections:
- net +5V: now also D5.C
- net N$37: now also D5.A
Changed lines of the file:
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@@
 <layer number="97" name="Info" color="7" fill="1" visible="yes" active="yes"/>
 <layer number="98" name="Guide" color="6" fill="1" visible="yes" active="yes"/>
+<layer number="99" name="SpiceOrder" color="5" fill="1" visible="yes" active="yes"/>
 </layers>
 <schematic xreflabel="%F%N/%S.%C%R" xrefpart="/%S.%C%R">
@@
 <part name="JP7" library="pinhead" deviceset="PINHD-1X4" device=""/>
 <part name="P+6" library="supply1" deviceset="+5V" device=""/>
+<part name="D5" library="diode" deviceset="1N4148" device="DO35-10"/>
 </parts>
 <sheets>
@@
 <instance part="JP7" gate="A" x="127" y="127"/>
 <instance part="P+6" gate="1" x="134.62" y="83.82" rot="R90"/>
+<instance part="D5" gate="G$1" x="200.66" y="58.42" rot="R270"/>
 </instances>
 <busses>
@@
 <pinref part="K1" gate="1" pin="2"/>
 <pinref part="P+10" gate="1" pin="+5V"/>
+<pinref part="D5" gate="G$1" pin="C"/>
+<wire x1="190.5" y1="53.34" x2="200.66" y2="53.34" width="0.1524" layer="91"/>
+<wire x1="200.66" y1="53.34" x2="200.66" y2="55.88" width="0.1524" layer="91"/>
+<junction x="190.5" y="53.34"/>
 </segment>
 <segment>
@@
 <wire x1="177.8" y1="66.04" x2="190.5" y2="66.04" width="0.1524" layer="91"/>
 <wire x1="190.5" y1="66.04" x2="190.5" y2="63.5" width="0.1524" layer="91"/>
-</segment>
-</net>
+<pinref part="D5" gate="G$1" pin="A"/>
+<wire x1="190.5" y1="66.04" x2="200.66" y2="66.04" width="0.1524" layer="91"/>
+<wire x1="200.66" y1="66.04" x2="200.66" y2="60.96" width="0.1524" layer="91"/>
+<junction x="190.5" y="66.04"/>
+</segment>
+</net>
